File: CopernicusBasicTestCircuit.sch (EAGLE design)
At the start: 6 parts, among them M1 COPERNICUS_II_MODULE

Commit message: Update schematic and pics
Connections:
- net N$2: now also U$1.D6; no longer U$1.D4
- net N$4: now also U$1.D5; no longer U$1.D3
Other:
- note added: "Rev 2.0.0 Far Horizons Lab May 27, 2014"
- note removed: "Rev 1.0 Far Horizons Lab Jan 20, 2014"
Changed lines of the file:
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@@
 <?xml version="1.0" encoding="utf-8"?>
 <!DOCTYPE eagle SYSTEM "eagle.dtd">
-<eagle version="6.4">
+<eagle version="6.5.0">
 <drawing>
 <settings>
@@
 <plain>
 <text x="38.1" y="127" size="3.81" layer="91">Trimble Copernicus II Sparkfun Module Basic Test Circuit</text>
-<text x="144.78" y="2.54" size="1.9304" layer="91">Software Serial
+<text x="144.78" y="7.62" size="1.9304" layer="91">Software Serial
 Assigned Pins</text>
-<text x="43.18" y="-12.7" size="1.778" layer="91">Rev 1.0
+<text x="43.18" y="-12.7" size="1.778" layer="91">Rev 2.0.0
 Far Horizons Lab
-Jan 20, 2014
+May 27, 2014
 </text>
 <text x="142.24" y="60.96" size="1.778" layer="91">Passive 5V to 3.3V
@@
 <segment>
 <pinref part="R1" gate="G$1" pin="2"/>
-<wire x1="165.1" y1="-2.54" x2="165.1" y2="71.12" width="0.1524" layer="91"/>
 <wire x1="165.1" y1="71.12" x2="152.4" y2="71.12" width="0.1524" layer="91"/>
-<pinref part="U$1" gate="G$1" pin="D3"/>
-<wire x1="139.7" y1="-2.54" x2="165.1" y2="-2.54" width="0.1524" layer="91"/>
+<wire x1="165.1" y1="71.12" x2="165.1" y2="2.54" width="0.1524" layer="91"/>
+<pinref part="U$1" gate="G$1" pin="D5"/>
+<wire x1="139.7" y1="2.54" x2="165.1" y2="2.54" width="0.1524" layer="91"/>
 </segment>
 </net>
@@
 <net name="N$2" class="0">
 <segment>
-<wire x1="170.18" y1="106.68" x2="170.18" y2="0" width="0.1524" layer="91"/>
+<wire x1="170.18" y1="106.68" x2="170.18" y2="5.08" width="0.1524" layer="91"/>
 <pinref part="R4" gate="G$1" pin="1"/>
 <pinref part="R3" gate="G$1" pin="2"/>
@@
 <wire x1="170.18" y1="106.68" x2="139.7" y2="106.68" width="0.1524" layer="91"/>
 <junction x="139.7" y="106.68"/>
-<pinref part="U$1" gate="G$1" pin="D4"/>
-<wire x1="139.7" y1="0" x2="170.18" y2="0" width="0.1524" layer="91"/>
-</segment>
-</net>
+<pinref part="U$1" gate="G$1" pin="D6"/>
+<wire x1="139.7" y1="5.08" x2="170.18" y2="5.08" width="0.1524" layer="91"/>
+</segment>
+</net>
